File: ESP32S3PCM5122/DAC-POWER.kicad_sch (KiCad schematic)
At the start: 9 parts, among them IC7 LT3042, IC8 TPS7A2033PDBVR

Commit message: more work
Parts:
- IC7: footprint Package_SO:MSOP-10-1EP_3x3mm_P0.5mm_EP1.68x1.88mm -> Custom:LT3042
- IC8: value TPS7A2033PDBVR -> TPS7A2033
Connections:
- net VBUS: now reaches C37.1, IC8.1 (IN), IC8.3 (EN)
- net VBUS: now also C34.1, C35.2, IC7.1 (IN_1), IC7.2 (IN_2), IC7.3 (EN/UV), IC7.6 (PGFB)
- net DAC3V3DIG: now reaches C38.1, IC8.5 (OUT)
- net DAC3V3ANA: now reaches C36.1, IC7.10 (OUT), IC7.9 (OUTS)
Changed lines of the file:
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@@
 	(wire
 		(pts
-			(xy 135.89 95.25) (xy 171.45 95.25)
+			(xy 135.89 95.25) (xy 170.18 95.25)
 		)
 		(stroke
@@
 	(wire
 		(pts
-			(xy 58.42 95.25) (xy 67.31 95.25)
-		)
-		(stroke
-			(width 0)
-			(type default)
-		)
-	)
-	(wire
-		(pts
 			(xy 129.54 102.87) (xy 129.54 81.28)
 		)
@@
 	(wire
 		(pts
+			(xy 44.45 41.91) (xy 72.39 41.91)
+		)
+		(stroke
+			(width 0)
+			(type default)
+		)
+	)
+	(wire
+		(pts
 			(xy 130.81 97.79) (xy 130.81 120.65)
 		)
@@
 	(wire
 		(pts
-			(xy 62.23 41.91) (xy 72.39 41.91)
-		)
-		(stroke
-			(width 0)
-			(type default)
-		)
-	)
-	(wire
-		(pts
 			(xy 135.89 120.65) (xy 135.89 107.95)
 		)
@@
 	(wire
 		(pts
-			(xy 128.27 44.45) (xy 149.86 44.45)
+			(xy 128.27 44.45) (xy 168.91 44.45)
 		)
 		(stroke
@@
 	(wire
 		(pts
+			(xy 44.45 95.25) (xy 67.31 95.25)
+		)
+		(stroke
+			(width 0)
+			(type default)
+		)
+	)
+	(wire
+		(pts
 			(xy 128.27 44.45) (xy 128.27 48.26)
 		)
@@
 			(width 0)
 			(type default)
+		)
+	)
+	(hierarchical_label "DAC3V3ANA"
+		(shape output)
+		(at 170.18 95.25 0)
+		(effects
+			(font
+				(size 1.27 1.27)
+			)
+			(justify left)
+		)
+	)
+	(hierarchical_label "VBUS"
+		(shape input)
+		(at 44.45 41.91 180)
+		(effects
+			(font
+				(size 1.27 1.27)
+			)
+			(justify right)
+		)
+	)
+	(hierarchical_label "VBUS"
+		(shape input)
+		(at 44.45 95.25 180)
+		(effects
+			(font
+				(size 1.27 1.27)
+			)
+			(justify right)
+		)
+	)
+	(hierarchical_label "DAC3V3DIG"
+		(shape output)
+		(at 168.91 44.45 0)
+		(effects
+			(font
+				(size 1.27 1.27)
+			)
+			(justify left)
 		)
 	)
@@
 			)
 		)
-		(property "Value" "TPS7A2033PDBVR"
+		(property "Value" "TPS7A2033"
 			(at 106.68 36.83 0)
 			(effects
@@
 			)
 		)
-		(property "Footprint" "Package_SO:MSOP-10-1EP_3x3mm_P0.5mm_EP1.68x1.88mm"
+		(property "Footprint" "Custom:LT3042"
 			(at 121.92 187.63 0)
 			(effects
