File: ESP32S3PCM5122/ESP32-POWER.kicad_sch (KiCad schematic)
At the start: 9 parts, among them IC2 AP63203

Commit message: more work
Changed lines of the file:
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@@
 		)
 	)
-	(global_label "ESP3V3"
+	(hierarchical_label "VBUS"
+		(shape input)
+		(at 71.12 73.66 180)
+		(effects
+			(font
+				(size 1.27 1.27)
+			)
+			(justify right)
+		)
+	)
+	(hierarchical_label "ESP3V3"
 		(shape output)
 		(at 224.79 71.12 0)
-		(fields_autoplaced yes)
 		(effects
 			(font
@@
 			(justify left)
 		)
-		(property "Intersheetrefs" "${INTERSHEET_REFS}"
-			(at 234.9113 71.12 0)
-			(effects
-				(font
-					(size 1.27 1.27)
-				)
-				(justify left)
-				(hide yes)
-			)
-		)
 	)
-	(global_label "VBUS"
-		(shape input)
-		(at 71.12 73.66 180)
-		(fields_autoplaced yes)
-		(effects
-			(font
-				(size 1.27 1.27)
-			)
-			(justify right)
-		)
-		(property "Intersheetrefs" "${INTERSHEET_REFS}"
-			(at 63.2362 73.66 0)
-			(effects
-				(font
-					(size 1.27 1.27)
-				)
-				(justify right)
-				(hide yes)
-			)
-		)
-	)
