File: ESP32S3PCM5122/USB-IN.kicad_sch (KiCad schematic)
At the start: 7 parts, among them IC4 USBLC6, J5 PWR SW, J7 USB IN

Commit message: more work
Changed lines of the file:
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@@
 		)
 	)
-	(global_label "D+"
+	(hierarchical_label "VBUS"
 		(shape output)
-		(at 86.36 72.39 180)
-		(fields_autoplaced yes)
+		(at 170.18 29.21 90)
+		(effects
+			(font
+				(size 1.27 1.27)
+			)
+			(justify left)
+		)
+	)
+	(hierarchical_label "D-"
+		(shape output)
+		(at 86.36 77.47 180)
 		(effects
 			(font
@@
 			(justify right)
 		)
-		(property "Intersheetrefs" "${INTERSHEET_REFS}"
-			(at 80.5324 72.39 0)
-			(effects
-				(font
-					(size 1.27 1.27)
-				)
-				(justify right)
-				(hide yes)
-			)
-		)
 	)
-	(global_label "VBUS"
+	(hierarchical_label "D+"
 		(shape output)
-		(at 170.18 29.21 90)
-		(fields_autoplaced yes)
-		(effects
-			(font
-				(size 1.27 1.27)
-			)
-			(justify left)
-		)
-		(property "Intersheetrefs" "${INTERSHEET_REFS}"
-			(at 170.18 21.3262 90)
-			(effects
-				(font
-					(size 1.27 1.27)
-				)
-				(justify left)
-				(hide yes)
-			)
-		)
-	)
-	(global_label "D-"
-		(shape output)
-		(at 86.36 77.47 180)
-		(fields_autoplaced yes)
+		(at 86.36 72.39 180)
 		(effects
 			(font
@@
 			(justify right)
 		)
-		(property "Intersheetrefs" "${INTERSHEET_REFS}"
-			(at 80.5324 77.47 0)
-			(effects
-				(font
-					(size 1.27 1.27)
-				)
-				(justify right)
-				(hide yes)
-			)
-		)
 	)
