File: ESP32S3PCM5122/ESP32.kicad_sch (KiCad schematic)
At the start: 11 parts, among them IC1 ESP32-S3-WROOM-1U-N16R8, IC3 RESET, IC5 BOOT, J2 VOL

Commit message: more
Parts:
- removed C11: 10uF, Capacitor_SMD:C_1206_3216Metric_Pad1.33x1.80mm_HandSolder, symbol Device:C
- added R26, R8, R9: 22R, Resistor_SMD:R_0805_2012Metric_Pad1.20x1.40mm_HandSolder, symbol Device:R
Connections:
- net BCK: now also R8.1
- net DATA: now also R9.1
- net LRCK: now also R26.1
- net at IC1.4 (IO4): now also R8.2
- net at IC1.5 (IO5): now also R9.2
- net at IC1.6 (IO6): now also R26.2
Other:
- moved on the sheet: C12
