File: ESP32S3PCM5122/ESP32S3PCM5122.kicad_sch (KiCad schematic)
At the start: 27 parts, among them IC1 ESP32-S3-WROOM-1U-N16R8, IC2 AP63203, IC4 USBLC6, J1 OUT, J2 VOL, J5 PWR SW, J6 PWR LED, J7 USB IN, U1 PCM5122PW

Commit message: move to PCM5242
Parts:
- removed C1: 470uF, Capacitor_THT:CP_Radial_D6.3mm_P2.50mm, symbol Device:C_Polarized
- removed C2, C3: 2n2, Capacitor_SMD:C_0805_2012Metric_Pad1.18x1.45mm_HandSolder, symbol Device:C
- removed C5: 10uF, Capacitor_SMD:C_1206_3216Metric_Pad1.33x1.80mm_HandSolder, symbol Device:C
- removed C6, C7: 100nF, Capacitor_SMD:C_1206_3216Metric_Pad1.33x1.80mm_HandSolder, symbol Device:C
- removed C8, C9: 22uF, Capacitor_SMD:C_0805_2012Metric_Pad1.18x1.45mm_HandSolder, symbol Device:C
- removed IC1: ESP32-S3-WROOM-1U-N16R8, Custom:ESP32S3WROOM1UN16R8, symbol Custom:ESP32-S3-WROOM-1U-N16R8
- removed IC2: AP63203, Custom:AP63205WU7, symbol Custom:AP63205WU-7
- removed IC4: USBLC6, Package_TO_SOT_SMD:SOT-23-6_Handsoldering, symbol Custom:USBLC6-2SC6
- removed J1: OUT, Connector_JST:JST_XH_B3B-XH-A_1x03_P2.50mm_Vertical, symbol Connector:Conn_01x03_Socket
- removed J5: PWR SW, Connector_JST:JST_XH_B2B-XH-A_1x02_P2.50mm_Vertical, symbol Connector:Conn_01x02_Socket
- removed J7: USB IN, Connector_JST:JST_XH_B6B-XH-A_1x06_P2.50mm_Vertical, symbol Connector:Conn_01x06_Socket
- removed L1: 3.9uH, Custom:SRR4528A-3R9Y, symbol Device:L
- removed R1, R2: 470R, Resistor_SMD:R_0805_2012Metric_Pad1.20x1.40mm_HandSolder, symbol Device:R
- removed R12, R13: 22R, Resistor_SMD:R_0805_2012Metric_Pad1.20x1.40mm_HandSolder, symbol Device:R
- removed R17, R18: 5K1, Resistor_SMD:R_0805_2012Metric_Pad1.20x1.40mm_HandSolder, symbol Device:R
- removed U1: PCM5122PW, Package_SO:TSSOP-28_4.4x9.7mm_P0.65mm, symbol Audio:PCM5122PW
- added J8: VOL BYPASS, Connector_JST:JST_XH_B2B-XH-A_1x02_P2.50mm_Vertical, symbol Connector:Conn_01x02_Socket
- added R5, R6, R7: 10K, Resistor_SMD:R_0603_1608Metric_Pad0.98x0.95mm_HandSolder, symbol Device:R
Connections:
- net 3V3DIG: now also R5.1, R6.1, R7.2
- net GND: now also J8.2 (Pin_2)
- new net EN: R5.2
- new net GPIO0: R6.2
- new net VOL-BYPASS: J8.1 (Pin_1), R7.1
Other:
- added sheet DAC (DAC.kicad_sch)
- added sheet DAC-POWER (DAC-POWER.kicad_sch)
- added sheet ES32-POWER (ESP32-POWER.kicad_sch)
- added sheet ESP32 (ESP32.kicad_sch)
- added sheet OPA1656-POWER (OPA1656-POWER.kicad_sch)
- added sheet USB-IN (USB-IN.kicad_sch)
- moved on the sheet: C10, J2, J6, R3, R4

Commit message: more work
Other:
- sheet DAC ports: added BCK, DAC3V3ANA, DAC3V3DIG, DATA, LRCK, SCK, SCL, SDA; removed none
- sheet DAC-POWER ports: added DAC3V3ANA, DAC3V3DIG, VBUS; removed none
- sheet ES32-POWER ports: added ESP3V3, VBUS; removed none
- sheet ESP32 ports: added 3V3ESP, BCK, D+, D-, DATA, LRCK, SCK, SCL, SDA; removed none
- sheet OPA1656-POWER ports: added VBUS; removed none
- sheet USB-IN ports: added D+, D-, VBUS; removed none

Commit message: more work
Parts:
- removed C10: 100nF, Capacitor_SMD:C_1206_3216Metric_Pad1.33x1.80mm_HandSolder, symbol Device:C
- removed J2: VOL, Connector_JST:JST_XH_B3B-XH-A_1x03_P2.50mm_Vertical, symbol Connector:Conn_01x03_Socket
- removed R4: 1K, Resistor_SMD:R_0805_2012Metric_Pad1.20x1.40mm_HandSolder, symbol Device:R
Other:
- sheet ESP32 ports: added VOLADC; removed none
