File: ESP32S3PCM5122/ESP32S3PCM5122.kicad_pcb (KiCad board)
At the start: 4 copper layers, 84 x 70 mm, 73 parts, among them IC1 ESP32-S3-WROOM-1U-N16R8, IC2 AP63203, IC3 RESET, IC4 USBLC6, IC5 BOOT, IC7 LT3042, IC8 TPS7A2033, J1 OUT, J2 VOL, J5 PWR SW, J6 PWR LED, J7 USB IN, J8 VOL BYPASS, U2 PCM5242, U3 OPA1656

Commit message: more
Parts:
- removed the C10 at (166.6, 134.4)
- removed the C10 at (252.9, 148.8)
- removed the R4 at (252.2, 154.9)
- removed R5, R6: 10K, Resistor_SMD:R_0603_1608Metric_Pad0.98x0.95mm_HandSolder
- added C10: 100nF, Capacitor_SMD:C_1206_3216Metric_Pad1.33x1.80mm_HandSolder, F.Cu at (166.6, 134.4)
- added R26: 22R, Resistor_SMD:R_0805_2012Metric_Pad1.20x1.40mm_HandSolder, F.Cu at (126.8, 120.9)
- added R8: 22R, Resistor_SMD:R_0805_2012Metric_Pad1.20x1.40mm_HandSolder, F.Cu at (126.8, 116.8)
- added R9: 22R, Resistor_SMD:R_0805_2012Metric_Pad1.20x1.40mm_HandSolder, F.Cu at (126.8, 118.9)
- C11: value 10uF -> 100nF
- moved R3 120.7 mm to (131.8, 144.3), turned to -90 degrees
- moved J6 114.3 mm to (125.3, 142.2)
- moved R7 104.4 mm to (143.6, 144.5), turned to -90 degrees
- moved C1 98.6 mm to (123.7, 88.8)
- moved J8 92.2 mm to (147.7, 142.2)
- moved C11 29.5 mm to (182.6, 116.8)
Connections:
- C11 pad 1: GND -> Net-(U2-LDOO)
- C11 pad 2: /ES32-POWER/ESP3V3 -> GND
- IC1 pad 4: unconnected-(IC1-IO4-Pad4) -> Net-(IC1-IO4)
- IC1 pad 5: unconnected-(IC1-IO5-Pad5) -> Net-(IC1-IO5)
- IC1 pad 6: unconnected-(IC1-IO6-Pad6) -> Net-(IC1-IO6)
- U2 pad 2: unconnected-(U2-LDOO-Pad2) -> Net-(U2-LDOO)
Routing:
- net /DAC/LRCK: track 0.00 -> 34.8 mm
- net /DAC/DATA: track 0.00 -> 31.8 mm
- net /DAC/BCK: track 0.00 -> 30.2 mm
- net Net-(IC1-IO5): track 0.00 -> 18.1 mm
- net Net-(IC1-IO4): track 0.00 -> 18.0 mm
- net Net-(IC1-IO6): track 0.00 -> 17.9 mm
- net /DAC-POWER/VBUS: track 141.4 -> 146.3 mm
- net /VOL-BYPASS: track 0.00 -> 4.67 mm
- net Net-(J6-Pin_2): track 0.00 -> 4.49 mm
- net GND: vias 94 -> 96
